Commit message: sdf servion 1.8 to 1.9

File: ros_gz_example_description/models/diffarm/diffarm.sdf.xacro (robot description, xacro)
@@ -1,4 +1,4 @@
 <?xml version="1.0" ?>
-<sdf version="1.8" xmlns:xacro="http://ros.org/wiki/xacro">
+<sdf version="1.9" xmlns:xacro="http://ros.org/wiki/xacro">
     <model name="diffarm" canonical_link="chassis">
         <xacro:property name="wheel_radius" value="0.4"/>
@@ -7,4 +7,5 @@
         <xacro:property name="chassis_y" value="1.0"/>
         <xacro:property name="chassis_z" value="0.5"/>
+        <xacro:property name="caster_radius" value="${wheel_radius/2}"/>
         <plugin
             filename="gz-sim-diff-drive-system"
@@ -148,5 +149,5 @@
 <!-- caster wheel -->
         <frame name="caster_frame" attached_to='chassis'>
-            <pose>0.8 0 -${wheel_radius/2} 0 0 0</pose>
+            <pose>${chassis_y-caster_radius} 0 -${caster_radius} 0 0 0</pose>
         </frame>
         <link name='caster'>
@@ -166,5 +167,5 @@
                 <geometry>
                     <sphere>
-                        <radius>${wheel_radius/2}</radius>
+                        <radius>${caster_radius}</radius>
                     </sphere>
                 </geometry>
@@ -178,5 +179,5 @@
                 <geometry>
                     <sphere>
-                        <radius>${wheel_radius/2}</radius>
+                        <radius>${caster_radius}</radius>
                     </sphere>
                 </geometry>

File: ros_gz_example_description/models/diffarm/ground_plane.sdf.xacro (robot description, xacro)
@@ -1,3 +1,3 @@
-<sdf version="1.8" xmlns:xacro="http://ros.org/wiki/xacro">
+<sdf version="1.9" xmlns:xacro="http://ros.org/wiki/xacro">
     <model name="ground_plane">
         <static>true</static>

File: ros_gz_example_description/models/diffarm/plugins.sdf.xacro (robot description, xacro)
@@ -1,4 +1,4 @@
 <?xml version="1.0" ?>
-<sdf version="1.8" xmlns:xacro="http://ros.org/wiki/xacro">
+<sdf version="1.9" xmlns:xacro="http://ros.org/wiki/xacro">
     <plugin
         filename="gz-sim-physics-system"

File: ros_gz_example_description/models/diffarm/wall.sdf.xacro (robot description, xacro)
@@ -1,4 +1,4 @@
 <?xml version="1.0" ?>
-<sdf version="1.8" xmlns:xacro="http://ros.org/wiki/xacro">
+<sdf version="1.9" xmlns:xacro="http://ros.org/wiki/xacro">
     <model name='wall'>
         <static>true</static>

File: ros_gz_example_description/models/diffarm/world.sdf.xacro (robot description, xacro)
@@ -1,5 +1,5 @@
 <?xml version="1.0" ?>
 <!-- this from "https://gazebosim.org/docs/garden/moving_robot" -->
-<sdf version="1.8" xmlns:xacro="http://ros.org/wiki/xacro">
+<sdf version="1.9" xmlns:xacro="http://ros.org/wiki/xacro">
     <world name="car_world">
         <physics name="1ms" type="ignored">

Commit message: add arm

File: ros_gz_example_description/models/diffarm/diffarm.sdf.xacro (robot description, xacro)
@@ -18,174 +18,8 @@
             <topic>cmd_vel</topic>
         </plugin>
-        <frame name="lidar_frame" attached_to='chassis'>
-            <pose>0.8 0 0.5 0 0 0</pose>
-        </frame>
-        <link name="chassis">
-            <pose relative_to="__model__">0.5 0 ${wheel_radius} 0 0 0</pose>
-            <inertial> <!--inertial properties of the link mass, inertia matix-->
-                <mass>1.14395</mass>
-                <inertia>
-                    <ixx>0.095329</ixx>
-                    <ixy>0</ixy>
-                    <ixz>0</ixz>
-                    <iyy>0.381317</iyy>
-                    <iyz>0</iyz>
-                    <izz>0.476646</izz>
-                </inertia>
-            </inertial>
-            <visual name='visual'>
-                <geometry>
-                    <box>
-                        <size>${chassis_x} ${chassis_y} ${chassis_z}</size>
-                    </box>
-                </geometry>
-                <!--let's add color to our link-->
-                <material>
-                    <ambient>0.0 0.0 1.0 1</ambient>
-                    <diffuse>0.0 0.0 1.0 1</diffuse>
-                    <specular>0.0 0.0 1.0 1</specular>
-                </material>
-            </visual>
-            <collision name='collision'>
-                <geometry>
-                    <box>
-                        <size>${chassis_x} ${chassis_y} ${chassis_z}</size>
-                    </box>
-                </geometry>
-            </collision>
-            <sensor name="imu_sensor" type="imu">
-                <always_on>1</always_on>
-                <update_rate>1</update_rate>
-                <visualize>true</visualize>
-                <topic>imu</topic>
-            </sensor>
-            <sensor name='gpu_lidar' type='gpu_lidar'>
-                <pose relative_to='lidar_frame'>0 0 0 0 0 0</pose>
-                <topic>lidar</topic>
-                <update_rate>10</update_rate>
-                <ray>
-                    <scan>
-                        <horizontal>
-                            <samples>640</samples>
-                            <resolution>1</resolution>
-                            <min_angle>-1.396263</min_angle>
-                            <max_angle>1.396263</max_angle>
-                        </horizontal>
-                        <vertical>
-                            <samples>1</samples>
-                            <resolution>0.01</resolution>
-                            <min_angle>0</min_angle>
-                            <max_angle>0</max_angle>
-                        </vertical>
-                    </scan>
-                    <range>
-                        <min>0.08</min>
-                        <max>10.0</max>
-                        <resolution>0.01</resolution>
-                    </range>
-                </ray>
-                <always_on>1</always_on>
-                <visualize>true</visualize>
-            </sensor>
-        </link>
-<!-- wheel -->
-        <xacro:macro name="wheel_link" params="prefix x y">
-          <link name='${prefix}_wheel'>
-            <pose relative_to="chassis">${x} ${y} 0 -1.5707 0 0</pose>
-              <inertial>
-                  <mass>1</mass>
-                  <inertia>
-                      <ixx>0.043333</ixx>
-                      <ixy>0</ixy>
-                      <ixz>0</ixz>
-                      <iyy>0.043333</iyy>
-                      <iyz>0</iyz>
-                      <izz>0.08</izz>
-                  </inertia>
-              </inertial>
-              <visual name='visual'>
-                <geometry>
-                    <cylinder>
-                        <radius>${wheel_radius}</radius>
-                        <length>${wheel_length}</length>
-                    </cylinder>
-                </geometry>
-                <material>
-                    <ambient>1.0 0.0 0.0 1</ambient>
-                    <diffuse>1.0 0.0 0.0 1</diffuse>
-                    <specular>1.0 0.0 0.0 1</specular>
-                </material>
-              </visual>
-              <collision name='collision'>
-                  <geometry>
-                      <cylinder>
-                          <radius>${wheel_radius}</radius>
-                          <length>${wheel_length}</length>
-                      </cylinder>
-                  </geometry>
-              </collision>
-          </link>
-        </xacro:macro> <!-- wheel -->
-        <xacro:macro name="wheel_joint" params="prefix">
-            <joint name='${prefix}_wheel_joint' type='continuous'>
-                <pose relative_to='${prefix}_wheel'/>
-                <parent>chassis</parent>
-                <child>${prefix}_wheel</child>
-                <axis>
-                    <xyz expressed_in='__model__'>0 1 0</xyz>
-                    <!-- <limit>
-                        <lower>-1.79769e+308</lower>
-                        <upper>1.79769e+308</upper>
-                    </limit> -->
-                </axis>
-            </joint>
-        </xacro:macro>  <!-- wheel_joint -->
-        <xacro:macro name="wheel" params="prefix x y">
-          <xacro:wheel_link prefix="${prefix}" x="${x}" y="${y}"/>
-          <xacro:wheel_joint prefix="${prefix}"/>
-        </xacro:macro>  <!-- wheel -->
-        <xacro:wheel prefix="left" x="-0.5" y="${(chassis_y+wheel_length)/2}"/>
-        <xacro:wheel prefix="right" x="-0.5" y="-${(chassis_y+wheel_length)/2}"/>
-<!-- caster wheel -->
-        <frame name="caster_frame" attached_to='chassis'>
-            <pose>${chassis_y-caster_radius} 0 -${caster_radius} 0 0 0</pose>
-        </frame>
-        <link name='caster'>
-            <pose relative_to='caster_frame'/>
-            <inertial>
-                <mass>1</mass>
-                <inertia>
-                    <ixx>0.016</ixx>
-                    <ixy>0</ixy>
-                    <ixz>0</ixz>
-                    <iyy>0.016</iyy>
-                    <iyz>0</iyz>
-                    <izz>0.016</izz>
-                </inertia>
-            </inertial>
-            <visual name='visual'>
-                <geometry>
-                    <sphere>
-                        <radius>${caster_radius}</radius>
-                    </sphere>
-                </geometry>
-                <material>
-                    <ambient>0.0 1 0.0 1</ambient>
-                    <diffuse>0.0 1 0.0 1</diffuse>
-                    <specular>0.0 1 0.0 1</specular>
-                </material>
-            </visual>
-            <collision name='collision'>
-                <geometry>
-                    <sphere>
-                        <radius>${caster_radius}</radius>
-                    </sphere>
-                </geometry>
-            </collision>
-        </link>
-        <joint name='caster_wheel' type='ball'>
-            <parent>chassis</parent>
-            <child>caster</child>
-        </joint>
+        <xacro:include filename="diffarm/chassis.sdf.xacro"/>
+        <xacro:include filename="diffarm/wheel.sdf.xacro"/>
+        <xacro:include filename="diffarm/caster_wheel.sdf.xacro"/>
+        <xacro:include filename="arm.sdf.xacro"/>
     </model>
 </sdf>
