Commit message: wheel joint "continuous" to "revolute"
because gazebo does not support "continuous" yet.

File: ros_gz_example_description/models/diffarm/diffarm/wheel.sdf.xacro (robot description, xacro)
@@ -39,5 +39,5 @@
     </xacro:macro> <!-- wheel_link -->
     <xacro:macro name="wheel_joint" params="prefix">
-        <joint name='${prefix}_wheel_joint' type='continuous'>
+        <joint name='${prefix}_wheel_joint' type='revolute'>
             <pose relative_to='${prefix}_wheel'/>
             <parent>chassis</parent>
@@ -45,8 +45,8 @@
             <axis>
                 <xyz expressed_in='__model__'>0 1 0</xyz>
-                <!-- <limit>
+                <limit>
                     <lower>-1.79769e+308</lower>
                     <upper>1.79769e+308</upper>
-                </limit> -->
+                </limit>
             </axis>
         </joint>
