Commit message: add temporary arm

File: ros_gz_example_description/models/diffarm/diffarm/arm.sdf.xacro (robot description, xacro)
@@ -41,9 +41,13 @@
           </collision>
       </link>
-      <joint name='arm_base_joint' type='continuous'>
+      <joint name='arm_base_joint' type='revolute'>
           <parent>chassis</parent>
           <child>arm_base</child>
           <axis>
-              <xyz expressed_in='__model__'>0 0 1</xyz>
+              <xyz>0 0 1</xyz>
+              <limit>
+                  <lower>-1.79769e+308</lower>
+                  <upper>1.79769e+308</upper>
+              </limit>
               <!-- <limit>
                   <lower>-1.79769e+308</lower>
@@ -52,48 +56,108 @@
           </axis>
       </joint>
-      <xacro:macro name="arm_stick" params="prefix parent">
-          <link name='${prefix}'>
-              <pose relative_to="${parent}">0 0 0 0 -0 0</pose>
-              <inertial>
-                  <pose>0 0 1 0 0 0</pose>
-                  <mass>1</mass>
-                  <inertia>
-                      <ixx>0.334167</ixx>
-                      <ixy>0</ixy>
-                      <ixz>0</ixz>
-                      <iyy>0.334167</iyy>
-                      <iyz>0</iyz>
-                      <izz>0.00166667</izz>
-                  </inertia>
-              </inertial>
-              <collision name='${prefix}_collision'>
-                  <pose>0 0 1 0 -0 0</pose>
-                  <geometry>
-                      <box>
-                          <size>0.1 0.1 2</size>
-                      </box>
-                  </geometry>
-              </collision>
-              <visual name='${prefix}_visual'>
-                  <pose>0 0 1 0 -0 0</pose>
-                  <geometry>
-                      <box>
-                          <size>0.1 0.1 2</size>
-                      </box>
-                  </geometry>
-                  <material>
-                      <diffuse> 1 0.423529412 0.039215686 1</diffuse>
-                      <ambient> 1 0.423529412 0.039215686 1</ambient>
-                      <specular>1 0.423529412 0.039215686 1</specular>
-                  </material>
-              </visual>
-          </link>
-      </xacro:macro>
-    <joint name='joint1' type='continuous'>
-      <pose relative_to='link1'>0 0.1 1.95 0 -0 0</pose>
-      <parent>link1</parent>
-      <child>link2</child>
+      <joint name='arm_first_joint' type='fixed'>
+        <parent>arm_base</parent>
+        <child>link1</child>
+      </joint>
+    <link name='link1'>
+      <pose relative_to="arm_base">0 0 0 0 -0 0</pose>
+      <inertial>
+        <pose>0 0 1 0 -0 0</pose>
+        <mass>1</mass>
+        <inertia>
+          <ixx>0.334167</ixx>
+          <ixy>0</ixy>
+          <ixz>0</ixz>
+          <iyy>0.334167</iyy>
+          <iyz>0</iyz>
+          <izz>0.00166667</izz>
+        </inertia>
+      </inertial>
+      <collision name='link1_collision'>
+        <pose>0 0 1 0 -0 0</pose>
+        <geometry>
+          <box>
+            <size>0.1 0.1 2</size>
+          </box>
+        </geometry>
+      </collision>
+      <visual name='link1_visual'>
+        <pose>0 0 1 0 -0 0</pose>
+        <geometry>
+          <box>
+            <size>0.1 0.1 2</size>
+          </box>
+        </geometry>
+        <material>
+          <diffuse> 1 0.423529412 0.039215686 1</diffuse>
+          <ambient> 1 0.423529412 0.039215686 1</ambient>
+          <specular>1 0.423529412 0.039215686 1</specular>
+        </material>
+      </visual>
+    </link>
+    <joint name='joint1' type='revolute'>
+        <pose relative_to='link1'>0 0.1 1.95 0 -0 0</pose>
+        <parent>link1</parent>
+        <child>link2</child>
+        <axis>
+            <xyz>0 1 0</xyz>
+            <limit>
+                <lower>-1.79769e+308</lower>
+                <upper>1.79769e+308</upper>
+            </limit>
+            <dynamics>
+              <damping>0.7</damping>
+              <friction>0.0</friction>
+              <spring_reference>0</spring_reference>
+              <spring_stiffness>0</spring_stiffness>
+            </dynamics>
+        </axis>
+    </joint>
+    <link name='link2'>
+      <pose relative_to='joint1'>0 0 0 0 -0 0</pose>
+      <inertial>
+        <pose>0 0 0.45 0 -0 0</pose>
+        <mass>1</mass>
+        <inertia>
+          <ixx>0.0841667</ixx>
+          <ixy>0</ixy>
+          <ixz>0</ixz>
+          <iyy>0.0841667</iyy>
+          <iyz>0</iyz>
+          <izz>0.00166667</izz>
+        </inertia>
+      </inertial>
+      <collision name='link2_collision'>
+        <pose>0 0 0.45 0 -0 0</pose>
+        <geometry>
+          <box>
+            <size>0.1 0.1 1</size>
+          </box>
+        </geometry>
+      </collision>
+      <visual name='link2_visual'>
+        <pose>0 0 0.45 0 -0 0</pose>
+        <geometry>
+          <box>
+            <size>0.1 0.1 1</size>
+          </box>
+        </geometry>
+        <material>
+          <diffuse> 0 0 0 1</diffuse>
+          <ambient> 0 0 0 1</ambient>
+          <specular>0 0 0 1</specular>
+        </material>
+      </visual>
+    </link>
+    <joint name='joint2' type='revolute'>
+      <pose relative_to='link2'>0 0.1 0.9 0 -0 0</pose>
+      <parent>link2</parent>
+      <child>link3</child>
       <axis>
         <xyz>0 1 0</xyz>
+        <limit>
+            <lower>-1.79769e+308</lower>
+            <upper>1.79769e+308</upper>
+        </limit>
         <dynamics>
           <damping>0.7</damping>
@@ -104,3 +168,39 @@
       </axis>
     </joint>
+    <link name='link3'>
+      <pose relative_to='joint2'>0 0 0 0 -0 0</pose>
+      <inertial>
+        <pose>0 0 0.45 0 -0 0</pose>
+        <mass>1</mass>
+        <inertia>
+          <ixx>0.0841667</ixx>
+          <ixy>0</ixy>
+          <ixz>0</ixz>
+          <iyy>0.0841667</iyy>
+          <iyz>0</iyz>
+          <izz>0.00166667</izz>
+        </inertia>
+      </inertial>
+      <collision name='link3_collision'>
+        <pose>0 0 0.45 0 -0 0</pose>
+        <geometry>
+          <box>
+            <size>0.1 0.1 1</size>
+          </box>
+        </geometry>
+      </collision>
+      <visual name='link3_visual'>
+        <pose>0 0 0.45 0 -0 0</pose>
+        <geometry>
+          <box>
+            <size>0.1 0.1 1</size>
+          </box>
+        </geometry>
+        <material>
+          <diffuse> 1 0.423529412 0.039215686 1</diffuse>
+          <ambient> 1 0.423529412 0.039215686 1</ambient>
+          <specular>1 0.423529412 0.039215686 1</specular>
+        </material>
+      </visual>
+    </link>
 </sdf>
